Commit message: kinda fixing the gps collision

File: urdf/sensors/gps.urdf.xacro (robot description, xacro)
@@ -13,7 +13,7 @@
       </visual>
       <collision>
-        <origin xyz="0 0 0.0324"/>
+        <origin xyz="0 0 0.0325"/>
         <geometry>
-          <sphere radius="0.1122"/>
+          <box size="0.152 0.152 0.065"/>
         </geometry>
       </collision>
