Commit message: fixing arm's camera mount and also gps

File: urdf/robot.urdf.xacro (robot description, xacro)
@@ -68,14 +68,46 @@
                         topic="/sensors/lidar3d_0/scan"
                         use_gazebo="$(arg use_gazebo)"/>
-  <!-- Wrist cameras (one per arm) and one neck camera -->
+  <!-- Wrist mounts + Fath pivots + RealSense cameras (one chain per arm) -->
+  <xacro:include filename="$(find husky_description)/urdf/accessories/wrist_mount.urdf.xacro"/>
+  <xacro:include filename="$(find husky_description)/urdf/accessories/fath_pivot_mount.urdf.xacro"/>
   <xacro:include filename="$(find husky_description)/urdf/sensors/realsense_d435.urdf.xacro"/>
-  <xacro:realsense_d435 prefix="camera_0" parent="arm_0_tool0"
-                        xyz="-0.08 0 0" rpy="0 -1.5708 0"
+  <!-- Left arm camera -->
+  <xacro:wrist_mount prefix="arm_0_wrist_mount" parent="arm_0_tool0"
+                    xyz="0 0 0" rpy="0 0 0"
+                    mesh_rpy="0 1.5708 -1.5708"/>
+  <!-- Alignment frame: lives in the rotated frame so children's poses stay valid -->
+  <link name="arm_0_wrist_mount_aligned"/>
+  <joint name="arm_0_wrist_mount_aligned_joint" type="fixed">
+    <parent link="arm_0_wrist_mount_link"/>
+    <child  link="arm_0_wrist_mount_aligned"/>
+    <origin xyz="0 0 0" rpy="0 1.5708 -1.5708"/>
+  </joint>
+  <xacro:fath_pivot_mount prefix="arm_0_pivot" parent="arm_0_wrist_mount_aligned"
+                          angle="${pi/12}"
+                          xyz="-0.01615 0 0.05842" rpy="0 0 3.14159"/>
+  <xacro:realsense_d435 prefix="camera_0" parent="arm_0_pivot_mount"
+                        xyz="0 0 0" rpy="0 0 0"
                         topic="/sensors/camera_0"
-                        use_gazebo="$(arg use_gazebo)"/>
-  <xacro:realsense_d435 prefix="camera_1" parent="arm_1_tool0"
-                        xyz="-0.08 0 0" rpy="0 -1.5708 0"
+                        use_gazebo="$(arg use_gazebo)"
+                        show_bracket="false"/>
+  <!-- Right arm camera -->
+  <xacro:wrist_mount prefix="arm_1_wrist_mount" parent="arm_1_tool0"
+                    xyz="0 0 0" rpy="0 0 0"
+                    mesh_rpy="0 1.5708 1.5708"/>
+  <!-- Alignment frame -->
+  <link name="arm_1_wrist_mount_aligned"/>
+  <joint name="arm_1_wrist_mount_aligned_joint" type="fixed">
+    <parent link="arm_1_wrist_mount_link"/>
+    <child  link="arm_1_wrist_mount_aligned"/>
+    <origin xyz="0 0 0" rpy="0 1.5708 1.5708"/>
+  </joint>
+  <xacro:fath_pivot_mount prefix="arm_1_pivot" parent="arm_1_wrist_mount_aligned"
+                          angle="${pi/12}"
+                          xyz="-0.01615 0 0.05842" rpy="0 0 3.14159"/>
+  <xacro:realsense_d435 prefix="camera_1" parent="arm_1_pivot_mount"
+                        xyz="0 0 0" rpy="0 0 0"
                         topic="/sensors/camera_1"
-                        use_gazebo="$(arg use_gazebo)"/>
+                        use_gazebo="$(arg use_gazebo)"
+                        show_bracket="false"/>
   <xacro:realsense_d435 prefix="camera_2" parent="neck_0_link"
                         xyz="0.01 0.0 -0.025" rpy="0 0 0"
@@ -92,5 +124,5 @@
   <xacro:include filename="$(find husky_description)/urdf/sensors/gps.urdf.xacro"/>
   <xacro:gps_sensor prefix="gps_0" parent="dual_arm_bulkhead_link"
-                    xyz="-0.20 0 0.19744" rpy="0 0 0"
+                    xyz="-0.20 0 0.27617" rpy="0 0 0"
                     topic="/sensors/gps_0/navsat"
                     use_gazebo="$(arg use_gazebo)"/>

File: urdf/sensors/gps.urdf.xacro (robot description, xacro)
@@ -1,19 +1,27 @@
 <?xml version="1.0"?>
-<!-- Swift GPS antenna macro. -->
+<!--
+  Swift Navigation GPS macro:
+    - ${prefix}_link        - Duro receiver (yellow box on parent)
+    - ${prefix}_antenna     - Swift antenna (white puck on top of receiver)
+  Two separate links because RViz has a long-standing bug where multiple
+  <visual> tags on a single link all get the first material's color.
+  See https://github.com/ros2/rviz/issues/1293
+-->
 <robot xmlns:xacro="http://www.ros.org/wiki/xacro">
   <xacro:macro name="gps_sensor"
                params="prefix parent xyz:='0 0 0' rpy:='0 0 0'
                        topic:='/navsat' use_gazebo:=false">
+    <!-- Receiver -->
     <link name="${prefix}_link">
       <visual>
-        <material name="clearpath_white"/>
+        <material name="clearpath_yellow"/>
         <geometry>
-          <mesh filename="package://husky_description/meshes/clearpath_sensors_description/meshes/swift_antenna.stl"/>
+          <mesh filename="package://husky_description/meshes/mount_description/duro_receiver.STL"/>
         </geometry>
       </visual>
       <collision>
-        <origin xyz="0 0 0.0325"/>
+        <origin xyz="0.013 0 -0.007" rpy="0 0 0"/>
         <geometry>
-          <box size="0.152 0.152 0.065"/>
+          <box size="0.152 0.152 0.144"/>
         </geometry>
       </collision>
@@ -23,4 +31,18 @@
       <parent link="${parent}"/>
       <child  link="${prefix}_link"/>
+    </joint>
+    <!-- Antenna sits at receiver's top face -->
+    <link name="${prefix}_antenna">
+      <visual>
+        <material name="clearpath_white"/>
+        <geometry>
+          <mesh filename="package://husky_description/meshes/clearpath_sensors_description/meshes/swift_antenna.stl"/>
+        </geometry>
+      </visual>
+    </link>
+    <joint name="${prefix}_antenna_joint" type="fixed">
+      <origin xyz="0 0 0" rpy="0 0 0"/>
+      <parent link="${prefix}_link"/>
+      <child  link="${prefix}_antenna"/>
     </joint>
     <xacro:if value="${use_gazebo}">
