Commit message: Swap lidar to VLP-32C, bake arm_0 hand-eye calibration, rework ZED Mini
Lidar: replace the VLP-16 macro with a VLP-32C Ultra Puck
(velodyne_vlp32c.urdf.xacro + VLP32C_base_1/base_2/scan meshes). Mount
pose, prefix and topic are unchanged, so lidar3d_0_link / lidar3d_0_laser
keep their frame names.

arm_0 hand-eye: the arm_0_wrist_mount joint now carries the measured
correction D = C * inv(N) (calibrated 2026-07-06). This moves the whole
bracket chain (wrist_mount -> aligned -> pivot -> bottom_screw ->
camera_link) as a rigid body, so camera_0 lands at its calibrated pose
while staying physically attached to the flange. arm_1 is still nominal
and needs the same treatment.

ZED Mini: replace the old prefix/parent macro with a local zed_mini macro
that reproduces the official zedm frame geometry and mesh but allows a
gray material (the upstream zed_camera macro hard-codes a
non-overridable black). Frame names match the ZED ROS 2 wrapper. The
neck attachment is now an explicit camera_2_mount_joint. Adds a
zed_description exec_depend for the mesh.

Known gap: the camera_2 mount offset is still an unmeasured estimate.

Co-Authored-By: Claude Opus 5 (1M context) <noreply@anthropic.com>
Claude-Session: https://claude.ai/code/session_014xVyFW1NxYb62mZeJX8vg2

File: urdf/robot.urdf.xacro (robot description, xacro)
@@ -62,17 +62,24 @@
   <!--  SENSORS                                                     -->
   <!-- =========================================================== -->
-  <!-- 3D Lidar on bulkhead -->
-  <xacro:include filename="$(find husky_description)/urdf/sensors/velodyne_vlp16.urdf.xacro"/>
-  <xacro:velodyne_vlp16 prefix="lidar3d_0" parent="dual_arm_bulkhead_link"
-                        xyz="0.35545 0.0 0.19744" rpy="0 0 0"
-                        topic="/sensors/lidar3d_0/scan"
-                        use_gazebo="$(arg use_gazebo)"/>
+  <!-- 3D Lidar on bulkhead (Velodyne VLP-32C Ultra Puck) -->
+  <xacro:include filename="$(find husky_description)/urdf/sensors/velodyne_vlp32c.urdf.xacro"/>
+  <xacro:velodyne_vlp32c prefix="lidar3d_0" parent="dual_arm_bulkhead_link"
+                         xyz="0.35545 0.0 0.19744" rpy="0 0 0"
+                         topic="/sensors/lidar3d_0/scan"
+                         use_gazebo="$(arg use_gazebo)"/>
   <!-- Wrist mounts + Fath pivots + RealSense cameras (one chain per arm) -->
   <xacro:include filename="$(find husky_description)/urdf/accessories/wrist_mount.urdf.xacro"/>
   <xacro:include filename="$(find husky_description)/urdf/accessories/fath_pivot_mount.urdf.xacro"/>
   <xacro:include filename="$(find husky_description)/urdf/sensors/realsense_d435.urdf.xacro"/>
-  <!-- Left arm camera -->
+  <!-- Left arm camera.
+       The wrist_mount joint carries the HAND-EYE CALIBRATION correction D = C * inv(N)
+       (2026-07-06), where N = nominal tool0->camera_0_link and C = measured. This
+       relocates the ENTIRE bracket (wrist_mount -> aligned -> pivot -> bottom_screw ->
+       camera_link) as a rigid body so the camera lands at the calibrated pose while
+       staying physically mounted to the bracket. The nominal chain was ~180 deg
+       mis-oriented; the correction is essentially a flip with ~0 translation, so the
+       bracket base stays on the flange and the assembly rotates to the true location. -->
   <xacro:wrist_mount prefix="arm_0_wrist_mount" parent="arm_0_tool0"
-                    xyz="0 0 0" rpy="0 0 0"
+                    xyz="-0.000107 0.004079 -0.033793" rpy="-0.072793 0.009861 3.130254"
                     mesh_rpy="0 1.5708 -1.5708"/>
   <!-- Alignment frame: lives in the rotated frame so children's poses stay valid -->
@@ -86,4 +93,7 @@
                           angle="${pi/12}"
                           xyz="-0.01615 0 0.05842" rpy="0 0 3.14159"/>
+  <!-- Camera rides the (now calibration-corrected) bracket: the wrist_mount joint
+       above carries the hand-eye correction, so this stays on the nominal pivot chain
+       and the camera + bracket move together (no floating camera). -->
   <xacro:realsense_d435 prefix="camera_0" parent="arm_0_pivot_mount"
                         xyz="0 0 0" rpy="0 0 0"
@@ -111,7 +121,18 @@
                         show_bracket="false"/>
 <!-- Neck ZED Mini camera (camera_2) -->
+  <!-- Local macro: EXACT official zedm frame geometry + official zed_description mesh,
+       but a gray material (official zed_camera macro hard-codes a black, non-overridable
+       material). Frame names match the ZED ROS 2 wrapper. -->
   <xacro:include filename="$(find husky_description)/urdf/sensors/zed_mini.urdf.xacro"/>
-  <xacro:zed_mini prefix="camera_2" parent="neck_0_link"
-                  xyz="0 0 0" rpy="0 0 0"/>
+  <xacro:zed_mini name="camera_2"/>
+  <!-- Mount: connect the ZED reference link (bottom screw hole) to the neck holder.
+       camera_2_camera_link is the manufacturer reference frame; everything below it
+       (camera_center, eyes, optical frames) is exact CAD and needs no tuning.
+       TODO: MEASURE this offset (neck_0_link -> ZED screw hole). Placeholder = identity. -->
+  <joint name="camera_2_mount_joint" type="fixed">
+    <parent link="neck_0_link"/>
+    <child  link="camera_2_camera_link"/>
+    <origin xyz="0.04 0.001 0.011" rpy="0 0 0"/>
+  </joint>
   <xacro:include filename="$(find husky_description)/urdf/sensors/imu.urdf.xacro"/>
   <xacro:imu_sensor prefix="imu_0" parent="base_link"

File: urdf/sensors/velodyne_vlp32c.urdf.xacro (robot description, xacro)
@@ -1,10 +1,19 @@
 <?xml version="1.0"?>
 <!--
-  Velodyne VLP-16 3D lidar macro.
-  Creates ${prefix}_link (sensor body) and ${prefix}_laser (optical frame).
+  Velodyne VLP-32C "Ultra Puck" 3D lidar macro.
+  Creates ${prefix}_link (sensor body) and ${prefix}_laser (scan/optical frame).
   Gazebo gpu_lidar plugin is added when use_gazebo:=true.
+  Note on the mesh: the VLP-32C shares the exact same external "Puck" housing as the
+  VLP-16 (103 mm diameter body) - the 32C just packs 32 laser pairs into the same
+  shell. The official velodyne_description ships no separate VLP-32C mesh for this
+  reason. The VLP32C_*.dae meshes here are the Puck body geometry (copied from the
+  VLP-16 Puck mesh) and are dimensionally correct for the VLP-32C body.
+  Real VLP-32C sensing differs from the VLP-16 and IS reflected in the <sensor> block:
+    - 32 vertical channels (vs 16)
+    - asymmetric vertical FOV +15 deg .. -25 deg = 40 deg total (vs +/-15 deg)
+    - up to 200 m range (vs 130 m)
 -->
 <robot xmlns:xacro="http://www.ros.org/wiki/xacro">
-  <xacro:macro name="velodyne_vlp16"
+  <xacro:macro name="velodyne_vlp32c"
                params="prefix parent xyz:='0 0 0' rpy:='0 0 0'
                        topic:='/scan' use_gazebo:=false">
@@ -12,5 +21,5 @@
     <link name="${prefix}_link">
       <inertial>
-        <mass value="0.83"/>
+        <mass value="0.925"/>  <!-- VLP-32C ~925 g (VLP-16 is 830 g) -->
         <origin xyz="0 0 0.03585"/>
         <inertia ixx="0.000908059425" ixy="0" ixz="0"
@@ -20,10 +29,10 @@
       <visual>
         <geometry>
-          <mesh filename="package://husky_description/meshes/velodyne_description/meshes/VLP16_base_1.dae"/>
+          <mesh filename="package://husky_description/meshes/velodyne_description/meshes/VLP32C_base_1.dae"/>
         </geometry>
       </visual>
       <visual>
         <geometry>
-          <mesh filename="package://husky_description/meshes/velodyne_description/meshes/VLP16_base_2.dae"/>
+          <mesh filename="package://husky_description/meshes/velodyne_description/meshes/VLP32C_base_2.dae"/>
         </geometry>
       </visual>
@@ -40,5 +49,5 @@
       <child  link="${prefix}_link"/>
     </joint>
-    <!-- Laser / optical frame -->
+    <!-- Laser / scan frame -->
     <link name="${prefix}_laser">
       <inertial>
@@ -52,5 +61,5 @@
         <origin xyz="0 0 -0.0377"/>
         <geometry>
-          <mesh filename="package://husky_description/meshes/velodyne_description/meshes/VLP16_scan.dae"/>
+          <mesh filename="package://husky_description/meshes/velodyne_description/meshes/VLP32C_scan.dae"/>
         </geometry>
       </visual>
@@ -61,9 +70,9 @@
       <child  link="${prefix}_laser"/>
     </joint>
-    <!-- Gazebo sensor plugin -->
+    <!-- Gazebo sensor plugin (VLP-32C: 32 channels, +15..-25 deg vertical, 200 m) -->
     <xacro:if value="${use_gazebo}">
       <gazebo reference="${prefix}_laser">
         <sensor name="${prefix}" type="gpu_lidar">
-          <update_rate>50</update_rate>
+          <update_rate>20</update_rate>  <!-- VLP-32C: 5-20 Hz -->
           <visualize>true</visualize>
           <always_on>true</always_on>
@@ -73,5 +82,5 @@
             <scan>
               <horizontal>
-                <samples>900</samples>
+                <samples>1800</samples>          <!-- ~0.2 deg azimuth resolution -->
                 <resolution>1</resolution>
                 <min_angle>-3.141592</min_angle>
@@ -79,13 +88,13 @@
               </horizontal>
               <vertical>
-                <samples>15</samples>
+                <samples>32</samples>
                 <resolution>1</resolution>
-                <min_angle>-0.261799</min_angle>
-                <max_angle> 0.261799</max_angle>
+                <min_angle>-0.436332</min_angle>  <!-- -25 deg -->
+                <max_angle> 0.261799</max_angle>  <!-- +15 deg -->
               </vertical>
             </scan>
             <range>
               <min>0.9</min>
-              <max>130.0</max>
+              <max>200.0</max>
               <resolution>0.01</resolution>
             </range>

File: urdf/sensors/zed_mini.urdf.xacro (robot description, xacro)
@@ -1,33 +1,81 @@
 <?xml version="1.0"?>
 <!--
-  Stereolabs ZED Mini stereo camera (neck camera_2).
-  Appearance/frames for RViz. Mesh is in METERS (scale 1 1 1).
-  Gazebo stereo sensor + optical frames can be added later behind use_gazebo.
+  ZED Mini (camera_2) - local macro.
+  Reproduces the EXACT frame geometry of Stereolabs' official zed_description
+  'zedm' model (constants copied verbatim from zed_macro.urdf.xacro):
+      baseline=0.063  height=0.0265  bottom_slope=0  optical_offset_x=0
+      screw_offset_x=0  screw_offset_z=0
+  Frame names and tree match the official wrapper exactly, so TF lines up with
+  the ZED ROS 2 node.
+  Why a local macro instead of <xacro:zed_camera>: the official macro hard-codes
+  a BLACK 'zedm_mat' material, and a URDF cannot redefine a material name
+  (urdfdom: "material 'zedm_mat' is not unique" -> fatal). This copy is identical
+  geometry but lets us pick the colour. The visual mesh still comes from the
+  installed zed_description package.
 -->
 <robot xmlns:xacro="http://www.ros.org/wiki/xacro">
-  <xacro:macro name="zed_mini"
-               params="prefix parent xyz:='0 0 0' rpy:='0 0 0'">
-    <!-- Mount frame: origin of the camera assembly on the holder -->
-    <joint name="${prefix}_joint" type="fixed">
-      <origin rpy="${rpy}" xyz="${xyz}"/>
-      <parent link="${parent}"/>
-      <child  link="${prefix}_link"/>
-    </joint>
-    <link name="${prefix}_link">
+  <material name="zed_gray"><color rgba="0.5 0.5 0.5 1.0"/></material>
+  <xacro:macro name="zed_mini" params="name">
+    <xacro:property name="baseline"         value="0.063"/>
+    <xacro:property name="height"           value="0.0265"/>
+    <xacro:property name="bottom_slope"     value="0.0"/>
+    <xacro:property name="optical_offset_x" value="0.0"/>
+    <xacro:property name="screw_offset_x"   value="0.0"/>
+    <xacro:property name="screw_offset_z"   value="0.0"/>
+    <!-- Mounting point (threaded screw hole in the bottom) -->
+    <link name="${name}_camera_link"/>
+    <!-- Camera body center (mesh lives here).
+         Visual uses the ORIGINAL official zed_description mesh, which is already
+         aligned to the camera_center frame (X-fwd, Y-left, Z-up), so no yaw/recenter
+         is needed (mesh origin = body center, like the official macro). VISUAL ONLY -
+         does not affect any TF/extrinsic. -->
+    <xacro:property name="mesh_rpy" value="0 0 0"/>
+    <xacro:property name="mesh_xyz" value="${screw_offset_x} 0 ${screw_offset_z}"/>
+    <link name="${name}_camera_center">
       <visual>
-        <origin rpy="0 0 -1.5708" xyz="0.031 0.0065 0.025"/>
+        <origin xyz="${mesh_xyz}" rpy="${mesh_rpy}"/>
         <geometry>
-          <mesh filename="package://husky_description/meshes/mount_description/ZEDM_bin.stl"
-                scale="1 1 1"/>
+          <mesh filename="package://zed_description/meshes/zedm.stl"/>
         </geometry>
-        <material name="clearpath_dark_grey"/>
+        <material name="zed_gray"/>
       </visual>
       <collision>
-        <origin rpy="0 0 -1.5708" xyz="0.031 0.0065 0.025"/>
+        <origin xyz="${mesh_xyz}" rpy="${mesh_rpy}"/>
         <geometry>
-          <box size="0.125 0.030 0.027"/>
+          <mesh filename="package://zed_description/meshes/zedm.stl"/>
         </geometry>
       </collision>
     </link>
+    <joint name="${name}_camera_center_joint" type="fixed">
+      <parent link="${name}_camera_link"/>
+      <child  link="${name}_camera_center"/>
+      <origin xyz="0 0 ${height/2}" rpy="0 ${bottom_slope} 0"/>
+    </joint>
+    <!-- Left camera -->
+    <link name="${name}_left_camera_frame"/>
+    <joint name="${name}_left_camera_joint" type="fixed">
+      <parent link="${name}_camera_center"/>
+      <child  link="${name}_left_camera_frame"/>
+      <origin xyz="${optical_offset_x} ${baseline/2} 0" rpy="0 0 0"/>
+    </joint>
+    <link name="${name}_left_camera_frame_optical"/>
+    <joint name="${name}_left_camera_optical_joint" type="fixed">
+      <parent link="${name}_left_camera_frame"/>
+      <child  link="${name}_left_camera_frame_optical"/>
+      <origin xyz="0 0 0" rpy="${-pi/2} 0 ${-pi/2}"/>
+    </joint>
+    <!-- Right camera -->
+    <link name="${name}_right_camera_frame"/>
+    <joint name="${name}_right_camera_joint" type="fixed">
+      <parent link="${name}_camera_center"/>
+      <child  link="${name}_right_camera_frame"/>
+      <origin xyz="${optical_offset_x} ${-baseline/2} 0" rpy="0 0 0"/>
+    </joint>
+    <link name="${name}_right_camera_frame_optical"/>
+    <joint name="${name}_right_camera_optical_joint" type="fixed">
+      <parent link="${name}_right_camera_frame"/>
+      <child  link="${name}_right_camera_frame_optical"/>
+      <origin xyz="0 0 0" rpy="${-pi/2} 0 ${-pi/2}"/>
+    </joint>
   </xacro:macro>
 </robot>
