Commit message: Swap neck camera

File: urdf/accessories/neck_camera_holder.urdf.xacro (robot description, xacro)
@@ -2,5 +2,5 @@
 <!--
   Neck camera holder - rigid bracket bolted to the FR12-H104 pan bracket.
-  Holds the 3rd RealSense D435 camera.
+  Holds the ZED camera.
 -->
 <robot xmlns:xacro="http://www.ros.org/wiki/xacro">
@@ -8,15 +8,15 @@
     <link name="${prefix}_link">
       <visual>
-        <origin rpy="-1.5708 0 1.5708" xyz="0 0 0"/>
+        <origin rpy="0 0 1.5708" xyz="0.0425 0.02 -0.01"/>
         <geometry>
-          <mesh filename="package://husky_description/meshes/mount_description/neck_camera_holder.stl"
+          <mesh filename="package://husky_description/meshes/mount_description/ZED_mount.stl"
                 scale="0.001 0.001 0.001"/>
         </geometry>
-        <material name="mount_olive_green"/>
+        <material name="clearpath_black"/>
       </visual>
       <collision>
-        <origin rpy="-1.5708 0 1.5708" xyz="0 0 0"/>
+        <origin rpy="0 0 1.5708" xyz="0.0425 0.02 -0.01"/>
         <geometry>
-          <mesh filename="package://husky_description/meshes/mount_description/neck_camera_holder.stl"
+          <mesh filename="package://husky_description/meshes/mount_description/ZED_mount.stl"
                 scale="0.001 0.001 0.001"/>
         </geometry>

File: urdf/robot.urdf.xacro (robot description, xacro)
@@ -45,5 +45,5 @@
   <!-- Neck camera holder -->
   <xacro:include filename="$(find husky_description)/urdf/accessories/neck_camera_holder.urdf.xacro"/>
-  <xacro:neck_camera_holder prefix="neck_0" parent="pan_0_link" xyz="0.038 -0.0025 0.034" rpy="0 0 0"/>
+  <xacro:neck_camera_holder prefix="neck_0" parent="pan_0_link" xyz="0 0 0" rpy="0 0 0"/>
   <!-- =========================================================== -->
   <!--  MANIPULATORS                                                -->
@@ -110,10 +110,8 @@
                         use_gazebo="$(arg use_gazebo)"
                         show_bracket="false"/>
-  <xacro:realsense_d435 prefix="camera_2" parent="neck_0_link"
-                        xyz="0.01 0.0 -0.025" rpy="0 0 0"
-                        topic="/sensors/camera_2"
-                        use_gazebo="$(arg use_gazebo)"
-                        show_bracket="false"/>
-  <!-- IMU -->
+<!-- Neck ZED Mini camera (camera_2) -->
+  <xacro:include filename="$(find husky_description)/urdf/sensors/zed_mini.urdf.xacro"/>
+  <xacro:zed_mini prefix="camera_2" parent="neck_0_link"
+                  xyz="0 0 0" rpy="0 0 0"/>
   <xacro:include filename="$(find husky_description)/urdf/sensors/imu.urdf.xacro"/>
   <xacro:imu_sensor prefix="imu_0" parent="base_link"
